Commit message: project2

File: src/my_robot/urdf/my_robot.xacro (robot description, xacro)
@@ -73,5 +73,5 @@
       <origin xyz="0 0 0" rpy="0 1.5707 1.5707"/>
       <geometry>
-        <cylinder radius="0.1" length="0.05"/>
+        <cylinder radius="0.2" length="0.05"/>
       </geometry>
     </collision>
@@ -79,5 +79,5 @@
       <origin xyz="0 0 0" rpy="0 1.5707 1.5707"/>
       <geometry>
-        <cylinder radius="0.1" length="0.05"/>
+        <cylinder radius="0.2" length="0.05"/>
       </geometry>
     </visual>
@@ -95,5 +95,5 @@
       <origin xyz="0 0 0" rpy="0 1.5707 1.5707"/>
       <geometry>
-        <cylinder radius="0.1" length="0.05"/>
+        <cylinder radius="0.2" length="0.05"/>
       </geometry>
     </collision>
@@ -101,6 +101,9 @@
       <origin xyz="0 0 0" rpy="0 1.5707 1.5707"/>
       <geometry>
-        <cylinder radius="0.1" length="0.05"/>
+        <cylinder radius="0.2" length="0.05"/>
       </geometry>
+      <material name ="red">
+      	<colour rgba="0.8 0.0 0.0 1.0"/>
+      </material>
     </visual>
   </link>

Commit message: Adjust wheel dimensions and add collision for visual

File: src/my_robot/urdf/my_robot.xacro (robot description, xacro)
@@ -73,5 +73,5 @@
       <origin xyz="0 0 0" rpy="0 1.5707 1.5707"/>
       <geometry>
-        <cylinder radius="0.2" length="0.05"/>
+        <cylinder radius="0.15" length="0.05"/>
       </geometry>
     </collision>
@@ -79,5 +79,5 @@
       <origin xyz="0 0 0" rpy="0 1.5707 1.5707"/>
       <geometry>
-        <cylinder radius="0.2" length="0.05"/>
+        <cylinder radius="0.15" length="0.05"/>
       </geometry>
     </visual>
@@ -95,5 +95,5 @@
       <origin xyz="0 0 0" rpy="0 1.5707 1.5707"/>
       <geometry>
-        <cylinder radius="0.2" length="0.05"/>
+        <cylinder radius="0.15" length="0.05"/>
       </geometry>
     </collision>
@@ -101,8 +101,8 @@
       <origin xyz="0 0 0" rpy="0 1.5707 1.5707"/>
       <geometry>
-        <cylinder radius="0.2" length="0.05"/>
+        <cylinder radius="0.15" length="0.05"/>
       </geometry>
       <material name ="red">
-      	<colour rgba="0.8 0.0 0.0 1.0"/>
+      	<color rgba="1 0 0 1"/>
       </material>
     </visual>
@@ -132,4 +132,10 @@
       </geometry>
     </visual>
+    <collision>
+      <origin xyz="0 0 0" rpy="0 0 0"/>
+      <geometry>
+        <box size="0.05 0.05 0.05"/>
+      </geometry>
+    </collision>
     <inertial>
       <mass value="0.1"/>

Commit message: project2

File: src/my_robot/urdf/my_robot.xacro (robot description, xacro)
@@ -2,4 +2,13 @@
 <robot name="my_robot" xmlns:xacro="http://www.ros.org/wiki/xacro">
 <xacro:include filename="$(find my_robot)/urdf/my_robot.gazebo" />
+  <material name="red">
+    <color rgba="1 0 0 1"/>
+  </material>
+  <material name="blue">
+    <color rgba="0 0 1 1"/>
+  </material>
+  <material name="dark_grey">
+    <color rgba="0.3 0.3 0.3 1"/>
+  </material>
   <!-- Base Footprint         -->
   <link name="robot_footprint"/>
@@ -32,4 +41,5 @@
         <box size="0.4 0.2 0.1"/>
       </geometry>
+      <material name="red"/>
     </visual>
     <!-- Back Caster -->
@@ -81,4 +91,5 @@
         <cylinder radius="0.15" length="0.05"/>
       </geometry>
+      <material name="blue"/>
     </visual>
   </link>
@@ -103,7 +114,5 @@
         <cylinder radius="0.15" length="0.05"/>
       </geometry>
-      <material name ="red">
-      	<color rgba="1 0 0 1"/>
-      </material>
+      <material name="blue"/>
     </visual>
   </link>
@@ -131,4 +140,5 @@
         <box size="0.05 0.05 0.05"/>
       </geometry>
+      <material name="dark_grey"/>
     </visual>
     <collision>

Commit message: project2

File: src/my_robot/urdf/my_robot.xacro (robot description, xacro)
@@ -47,5 +47,5 @@
       <origin xyz="-0.15 0 -0.05" rpy="0 0 0"/>
       <geometry>
-        <sphere radius="0.0499"/>
+        <sphere radius="0.1"/>
       </geometry>
     </collision>
@@ -53,5 +53,5 @@
       <origin xyz="-0.15 0 -0.05" rpy="0 0 0"/>
       <geometry>
-        <sphere radius="0.05"/>
+        <sphere radius="0.1"/>
       </geometry>
     </visual>
@@ -60,5 +60,5 @@
       <origin xyz="0.15 0 -0.05" rpy="0 0 0"/>
       <geometry>
-        <sphere radius="0.0499"/>
+        <sphere radius="0.1"/>
       </geometry>
     </collision>
@@ -66,5 +66,5 @@
       <origin xyz="0.15 0 -0.05" rpy="0 0 0"/>
       <geometry>
-        <sphere radius="0.05"/>
+        <sphere radius="0.1"/>
       </geometry>
     </visual>

Commit message: course5

File: src/my_robot/urdf/my_robot.xacro (robot description, xacro)
@@ -162,4 +162,11 @@
     <axis xyz="0 1 0"/>
   </joint>
+  <joint name="camera_optical_joint" type="fixed">
+    <origin xyz="0 0 0" rpy="-1.5707 0 -1.5707"/>
+    <parent link="camera"/>
+    <child link="camera_link_optical"/>
+  </joint>
+  <link name="camera_link_optical">
+  </link>
   <!-- Hokuyo Link -->
     <link name="hokuyo">
