Commit message: updated dependencies

File: src/kobuki_description/urdf/kobuki.urdf.xacro (robot description, xacro)
@@ -7,8 +7,6 @@
  -->
 <robot name="kobuki" xmlns:xacro="http://ros.org/wiki/xacro">
-  <include filename="$(find kobuki_description)/urdf/common_properties.urdf.xacro"/>
-  <include filename="$(find kobuki_description)/urdf/kobuki_gazebo.urdf.xacro"/>
-  <!-- Xacro properties -->
-  <xacro:property name="M_SCALE" value="0.001"/>
+  <xacro:include filename="$(find kobuki_description)/urdf/common_properties.urdf.xacro"/>
+  <xacro:include filename="$(find kobuki_description)/urdf/kobuki_gazebo.urdf.xacro"/>
   <!-- Kobuki -->
   <xacro:macro name="kobuki">
@@ -36,16 +34,24 @@
         <origin xyz="0.001 0 0.05199" rpy="0 0 0"/>
       </visual>
-      <collision>
-        <geometry>
-          <cylinder length="0.10938" radius="0.176"/>
+      <collision name="base">
+        <geometry>
+          <cylinder length="0.10938" radius="0.178"/>
         </geometry>
         <origin xyz="0.0 0 0.05949" rpy="0 0 0"/>
       </collision>
       <inertial>
+        <!-- COM experimentally determined -->
+        <origin xyz="0.01 0 0"/>
         <mass value="2.4"/> <!-- 2.4/2.6 kg for small/big battery pack -->
-        <origin xyz="0 0 0"/>
-        <inertia ixx="0.0001" ixy="0.0" ixz="0.0"
-                 iyy="0.0001" iyz="0.0"
-                 izz="0.0001" />
+        <!-- Kobuki's inertia tensor is approximated by a cylinder with homogeneous mass distribution
+             More details: http://en.wikipedia.org/wiki/List_of_moment_of_inertia_tensors
+             m = 2.4 kg; h = 0.09 m; r = 0.175 m
+             ixx = 1/12 * m * (3 * r^2 + h^2)
+             iyy = 1/12 * m * (3 * r^2 + h^2)
+             izz = 1/2 * m * r^2
+          -->
+        <inertia ixx="0.019995" ixy="0.0" ixz="0.0"
+                 iyy="0.019995" iyz="0.0"
+                 izz="0.03675" />
       </inertial>
     </link>
@@ -65,5 +71,5 @@
       <collision>
         <geometry>
-          <cylinder length="0.0206" radius="0.0352"/>
+          <cylinder length="0.0206" radius="0.035"/>
         </geometry>
         <origin rpy="0 0 0" xyz="0 0 0"/>
@@ -92,5 +98,5 @@
       <collision>
         <geometry>
-          <cylinder length="0.0206" radius="0.0350"/>
+          <cylinder length="0.0206" radius="0.035"/>
         </geometry>
         <origin rpy="0 0 0" xyz="0 0 0"/>
@@ -160,10 +166,10 @@
       </inertial>
     </link>
-	  <joint name="cliff_sensor_left_joint" type="fixed">
-	    <origin xyz="0.08734 0.13601 0.0214" rpy="0 ${M_PI/2} 0" />
-	    <parent link="base_link"/>
-	    <child link="cliff_sensor_left_link" />
-	  </joint>
-	  <link name="cliff_sensor_left_link">
+    <joint name="cliff_sensor_left_joint" type="fixed">
+      <origin xyz="0.08734 0.13601 0.0214" rpy="0 ${M_PI/2} 0" />
+      <parent link="base_link"/>
+      <child link="cliff_sensor_left_link" />
+    </joint>
+    <link name="cliff_sensor_left_link">
       <inertial>
         <mass value="0.0001" />
@@ -174,9 +180,9 @@
       </inertial>
     </link>
-	  <joint name="cliff_sensor_right_joint" type="fixed">
-	    <origin xyz="0.085 -0.13601 0.0214" rpy="0 ${M_PI/2} 0" />
-	    <parent link="base_link"/>
-	    <child link="cliff_sensor_right_link" />
-	  </joint>
+    <joint name="cliff_sensor_right_joint" type="fixed">
+      <origin xyz="0.085 -0.13601 0.0214" rpy="0 ${M_PI/2} 0" />
+      <parent link="base_link"/>
+      <child link="cliff_sensor_right_link" />
+    </joint>
     <link name="cliff_sensor_right_link">
       <inertial>
@@ -202,9 +208,6 @@
       </inertial>
     </link>
-    <!--  Gazebo additions -->
-    <kobuki_sim/>
-    <kobuki_bumpers/>
-    <kobuki_cliff_sensors/>
-    <kobuki_sim_imu/>
+    <!-- Kobuki Gazebo simulation details -->
+    <xacro:kobuki_sim/>
   </xacro:macro>
 </robot>

File: src/kobuki_description/urdf/kobuki_gazebo.urdf.xacro (robot description, xacro)
@@ -1,117 +1,198 @@
 <?xml version="1.0"?>
-<robot xmlns:controller="http://playerstage.sourceforge.net/gazebo/xmlschema/#controller"
-       xmlns:interface="http://playerstage.sourceforge.net/gazebo/xmlschema/#interface"
-       xmlns:sensor="http://playerstage.sourceforge.net/gazebo/xmlschema/#sensor"
-       xmlns:xacro="http://ros.org/wiki/xacro"
-       name="kobuki_gazebo">
-<xacro:macro name="kobuki_bumpers">
-  <gazebo reference="base_link">
-    <sensor:contact name="bumpers">
-      <geom>base_footprint_geom_base_link</geom>
-      <topic>bumpers</topic>
-      <alwaysOn>true</alwaysOn>
-      <updateRate>50</updateRate>
-    </sensor:contact>
-  </gazebo>
-</xacro:macro>
-<xacro:macro name="kobuki_cliff_sensors">
-  <gazebo reference="cliff_sensor_left_link">
-    <sensor:ray name="cliff_sensor_left">
-      <alwaysOn>true</alwaysOn>
-      <updateRate>50</updateRate>
-      <rayCount>50</rayCount>
-      <rangeCount>1</rangeCount>
-      <resRange>1.0</resRange>
-      <minAngle>-0.04361</minAngle>
-      <maxAngle>0.04361</maxAngle>
-      <minRange>0.01</minRange>
-      <maxRange>0.15</maxRange>
-      <displayRays>true</displayRays>
-    </sensor:ray>
-  </gazebo>
-  <gazebo reference="cliff_sensor_right_link">
-    <sensor:ray name="cliff_sensor_right">
-      <alwaysOn>true</alwaysOn>
-      <updateRate>50</updateRate>
-      <rayCount>50</rayCount>
-      <rangeCount>1</rangeCount>
-      <resRange>1.0</resRange>
-      <minAngle>-2.5</minAngle>
-      <maxAngle>2.5</maxAngle>
-      <minRange>0.01</minRange>
-      <maxRange>0.15</maxRange>
-      <displayRays>true</displayRays>
-    </sensor:ray>
-  </gazebo>
-  <gazebo reference="cliff_sensor_front_link">
-    <sensor:ray name="cliff_sensor_front">
-      <alwaysOn>true</alwaysOn>
-      <updateRate>50</updateRate>
-      <rayCount>50</rayCount>
-      <rangeCount>1</rangeCount>
-      <resRange>1.0</resRange>
-      <minAngle>-2.5</minAngle>
-      <maxAngle>2.5</maxAngle>
-      <minRange>0.01</minRange>
-      <maxRange>0.15</maxRange>
-      <displayRays>true</displayRays>
-    </sensor:ray>
-  </gazebo>
-</xacro:macro>
-<xacro:macro name="kobuki_sim">
-  <gazebo>
-    <controller:gazebo_ros_kobuki name="kobuki_controller" plugin="libgazebo_ros_kobuki.so">
-      <left_wheel_joint_name>wheel_left_joint</left_wheel_joint_name>
-      <right_wheel_joint_name>wheel_right_joint</right_wheel_joint_name>
-      <wheel_separation>.230</wheel_separation>
-      <wheel_diameter>0.070</wheel_diameter>
-      <torque>1.0</torque>
-      <velocity_command_timeout>0.6</velocity_command_timeout>
-      <cliff_sensor_left_name>cliff_sensor_left</cliff_sensor_left_name>
-      <cliff_sensor_front_name>cliff_sensor_front</cliff_sensor_front_name>
-      <cliff_sensor_right_name>cliff_sensor_right</cliff_sensor_right_name>
-      <cliff_detection_threshold>0.04</cliff_detection_threshold>
-      <bumper_name>bumpers</bumper_name>
-      <base_collision_model_link>base_link</base_collision_model_link>
-    </controller:gazebo_ros_kobuki>
-  </gazebo>
-  <gazebo reference="wheel_left_link">
-    <mu1 value="10"/>
-    <mu2 value="10"/>
-    <kp value="100000000.0"/>
-    <kd value="10000.0"/>
-  </gazebo>
-  <gazebo reference="wheel_right_link">
-    <mu1 value="10"/>
-    <mu2 value="10"/>
-    <kp value="100000000.0"/>
-    <kd value="10000.0"/>
-  </gazebo>
-  <gazebo reference="caster_front_link">
-    <mu1 value="0"/>
-    <mu2 value="0"/>
-    <kp value="100000000.0"/>
-    <kd value="10000.0"/>
-  </gazebo>
-  <gazebo reference="caster_back_link">
-    <mu1 value="0"/>
-    <mu2 value="0"/>
-    <kp value="100000000.0"/>
-    <kd value="10000.0"/>
-  </gazebo>
-</xacro:macro>
-<xacro:macro name="kobuki_sim_imu">
-  <gazebo>
-    <controller:gazebo_ros_imu name="imu_controller" plugin="libgazebo_ros_imu.so">
-      <alwaysOn>true</alwaysOn>
-      <updateRate>50</updateRate>
-      <bodyName>gyro_link</bodyName>
-      <topicName>/mobile_base/sensors/imu_data</topicName>
-      <gaussianNoise>${0.0017*0.0017}</gaussianNoise>
-      <xyzOffsets>0 0 0</xyzOffsets>
-      <rpyOffsets>0 0 0</rpyOffsets>
-      <interface:position name="gyro_link"/>
-    </controller:gazebo_ros_imu>
-  </gazebo>
-</xacro:macro>
+<robot name="kobuki_sim" xmlns:xacro="http://ros.org/wiki/xacro">
+  <xacro:macro name="kobuki_sim">
+    <gazebo reference="wheel_left_link">
+      <mu1>1.0</mu1>
+      <mu2>1.0</mu2>
+      <kp>1000000.0</kp>
+      <kd>100.0</kd>
+      <minDepth>0.001</minDepth>
+      <maxVel>1.0</maxVel>
+      <sensor type="contact" name="wheel_drop_left">
+        <always_on>1</always_on>
+        <update_rate>50.0</update_rate>
+        <visualize>true</visualize>
+        <contact>
+          <collision>wheel_left_link_collision</collision>
+        </contact>
+      </sensor>
+    </gazebo>
+    <gazebo reference="wheel_right_link">
+      <mu1>1.0</mu1>
+      <mu2>1.0</mu2>
+      <kp>1000000.0</kp>
+      <kd>100.0</kd>
+      <minDepth>0.001</minDepth>
+      <maxVel>1.0</maxVel>
+      <sensor type="contact" name="wheel_drop_right">
+        <always_on>1</always_on>
+        <update_rate>50.0</update_rate>
+        <visualize>true</visualize>
+        <contact>
+          <collision>wheel_right_link_collision</collision>
+        </contact>
+      </sensor>
+    </gazebo>
+    <gazebo reference="caster_front_link">
+      <mu1>0.0</mu1>
+      <mu2>0.0</mu2>
+      <kp>1000000.0</kp>
+      <kd>100.0</kd>
+      <minDepth>0.001</minDepth>
+      <maxVel>1.0</maxVel>
+    </gazebo>
+    <gazebo reference="caster_back_link">
+      <mu1>0.0</mu1>
+      <mu2>0.0</mu2>
+      <kp>1000000.0</kp>
+      <kd>100.0</kd>
+      <minDepth>0.001</minDepth>
+      <maxVel>1.0</maxVel>
+    </gazebo>
+    <gazebo reference="base_link">
+      <mu1>0.3</mu1>
+      <mu2>0.3</mu2>
+      <sensor type="contact" name="bumpers">
+        <always_on>1</always_on>
+        <update_rate>50.0</update_rate>
+        <visualize>true</visualize>
+        <contact>
+          <collision>base_footprint_fixed_joint_lump__base_collision</collision>
+        </contact>
+      </sensor>
+    </gazebo>
+    <gazebo reference="cliff_sensor_left_link">
+      <sensor type="ray" name="cliff_sensor_left">
+        <always_on>true</always_on>
+        <update_rate>50</update_rate>
+        <visualize>true</visualize>
+        <ray>
+          <scan>
+            <horizontal>
+              <samples>50</samples>
+              <resolution>1.0</resolution>
+              <min_angle>-0.0436</min_angle>  <!-- -2.5 degree -->
+              <max_angle>0.0436</max_angle> <!-- 2.5 degree -->
+            </horizontal>
+<!--            Can't use vertical rays until this bug is resolved: -->
+<!--            https://bitbucket.org/osrf/gazebo/issue/509/vertical-sensor-doesnt-works -->
+<!--               <vertical> -->
+<!--                 <samples>50</samples> -->
+<!--                 <resolution>1.0</resolution> -->
+<!--                 <min_angle>-0.0436</min_angle>  -2.5 degree -->
+<!--                 <max_angle>0.0436</max_angle> 2.5 degree -->
+<!--               </vertical> -->
+          </scan>
+          <range>
+            <min>0.01</min>
+            <max>0.15</max>
+            <resolution>1.0</resolution>
+          </range>
+        </ray>
+      </sensor>
+    </gazebo>
+    <gazebo reference="cliff_sensor_right_link">
+      <sensor type="ray" name="cliff_sensor_right">
+        <always_on>true</always_on>
+        <update_rate>50</update_rate>
+        <visualize>true</visualize>
+        <ray>
+          <scan>
+            <horizontal>
+              <samples>50</samples>
+              <resolution>1.0</resolution>
+              <min_angle>-0.0436</min_angle>  <!-- -2.5 degree -->
+              <max_angle>0.0436</max_angle> <!-- 2.5 degree -->
+            </horizontal>
+<!--            Can't use vertical rays until this bug is resolved: -->
+<!--            https://bitbucket.org/osrf/gazebo/issue/509/vertical-sensor-doesnt-works -->
+<!--               <vertical> -->
+<!--                 <samples>50</samples> -->
+<!--                 <resolution>1.0</resolution> -->
+<!--                 <min_angle>-0.0436</min_angle>  -2.5 degree -->
+<!--                 <max_angle>0.0436</max_angle> 2.5 degree -->
+<!--               </vertical> -->
+          </scan>
+          <range>
+            <min>0.01</min>
+            <max>0.15</max>
+            <resolution>1.0</resolution>
+          </range>
+        </ray>
+      </sensor>
+    </gazebo>
+    <gazebo reference="cliff_sensor_front_link">
+      <sensor type="ray" name="cliff_sensor_front">
+        <always_on>true</always_on>
+        <update_rate>50</update_rate>
+        <visualize>true</visualize>
+        <ray>
+          <scan>
+            <horizontal>
+              <samples>50</samples>
+              <resolution>1.0</resolution>
+              <min_angle>-0.0436</min_angle>  <!-- -2.5 degree -->
+              <max_angle>0.0436</max_angle> <!-- 2.5 degree -->
+            </horizontal>
+<!--               Can't use vertical rays until this bug is resolved: -->
+<!--            https://bitbucket.org/osrf/gazebo/issue/509/vertical-sensor-doesnt-works -->
+<!--               <vertical> -->
+<!--                 <samples>50</samples> -->
+<!--                 <resolution>1.0</resolution> -->
+<!--                 <min_angle>-0.0436</min_angle>  -2.5 degree -->
+<!--                 <max_angle>0.0436</max_angle> 2.5 degree -->
+<!--               </vertical> -->
+          </scan>
+          <range>
+            <min>0.01</min>
+            <max>0.15</max>
+            <resolution>1.0</resolution>
+          </range>
+        </ray>
+      </sensor>
+    </gazebo>
+    <gazebo reference="gyro_link">
+      <sensor type="imu" name="imu">
+      <always_on>true</always_on>
+      <update_rate>50</update_rate>
+      <visualize>false</visualize>
+      <imu>
+          <noise>
+            <type>gaussian</type>
+            <rate>
+              <mean>0.0</mean>
+              <stddev>${0.0014*0.0014}</stddev> <!-- 0.25 x 0.25 (deg/s) -->
+              <bias_mean>0.0</bias_mean>
+              <bias_stddev>0.0</bias_stddev>
+            </rate>
+            <accel> <!-- not used in the plugin and real robot, hence using tutorial values -->
+              <mean>0.0</mean>
+              <stddev>1.7e-2</stddev>
+              <bias_mean>0.1</bias_mean>
+              <bias_stddev>0.001</bias_stddev>
+            </accel>
+          </noise>
+        </imu>
+      </sensor>
+    </gazebo>
+    <gazebo>
+      <plugin name="kobuki_controller" filename="libgazebo_ros_kobuki.so">
+        <publish_tf>1</publish_tf>
+        <left_wheel_joint_name>wheel_left_joint</left_wheel_joint_name>
+        <right_wheel_joint_name>wheel_right_joint</right_wheel_joint_name>
+        <wheel_separation>.230</wheel_separation>
+        <wheel_diameter>0.070</wheel_diameter>
+        <torque>1.0</torque>
+        <velocity_command_timeout>0.6</velocity_command_timeout>
+        <cliff_sensor_left_name>cliff_sensor_left</cliff_sensor_left_name>
+        <cliff_sensor_center_name>cliff_sensor_front</cliff_sensor_center_name>
+        <cliff_sensor_right_name>cliff_sensor_right</cliff_sensor_right_name>
+        <cliff_detection_threshold>0.04</cliff_detection_threshold>
+        <bumper_name>bumpers</bumper_name>
+        <imu_name>imu</imu_name>
+        <wheel_drop_left_sensor_name>wheel_drop_left</wheel_drop_left_sensor_name>
+        <wheel_drop_right_sensor_name>wheel_drop_right</wheel_drop_right_sensor_name>
+      </plugin>
+    </gazebo>
+  </xacro:macro>
 </robot>

File: src/kobuki_description/urdf/kobuki_standalone.urdf.xacro (robot description, xacro)
@@ -6,5 +6,5 @@
        xmlns:xacro="http://ros.org/wiki/xacro">
   <!-- Defines the kobuki component tag. -->
-  <include filename="$(find kobuki_description)/urdf/kobuki.urdf.xacro" />
-  <kobuki/>
+  <xacro:include filename="$(find kobuki_description)/urdf/kobuki.urdf.xacro" />
+  <xacro:kobuki/>
 </robot>
